File: pcb/keyboard_l.kicad_sch (KiCad schematic)
At the start: 74 parts, among them J2 USB_C_Receptacle_USB2.0_16P, M1 Motor 2 +, M2 Motor 2 -, M3 Motor 1 -, M4 Motor 1 +, Q1 AO3400A

Commit message: Initial PCB v1.1.0 updates, including 4-layer restructure
Parts:
- added H12: Mounting_Hole, MountingHole:MountingHole_4.3mm_M4, symbol ScottoKeebs:Placeholder_Mounting_Hole
- added S41: SSAG230400, SSAG230400:SSAG230400, symbol SSAG230400:SSAG230400
Connections:
- net 5v L: now also S41.3 (COM); no longer M1.1, M4.1
- new net: M1.1, M4.1, S41.1 (NO_1)
- no-connect marks 5 -> 8
Other:
- moved on the sheet: D26, M1, M2, M3, M4, Q1, R6, R7

Commit message: Include components as a path in the repository
Parts:
- S1, S10, S11, S12, S13, S14, S15, S16, S17, S18, S19, S2, S20, S3, S4, S5, S6, S7, S9: footprint JacobGable:MX_Choc_Hotswap_Hybrid -> AlphaCentauri:MX_Choc_Hotswap_Hybrid
- S8: footprint JacobGable:MX_Choc_Hotswap_Hybrid_1.5u -> AlphaCentauri:MX_Choc_Hotswap_Hybrid_1.5u
Changed lines of the file:
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@@
 			)
 		)
-		(property "Footprint" "JacobGable:MX_Choc_Hotswap_Hybrid"
+		(property "Footprint" "AlphaCentauri:MX_Choc_Hotswap_Hybrid"
 			(at 259.08 156.21 0)
 			(hide yes)
@@
 			)
 		)
-		(property "Footprint" "JacobGable:MX_Choc_Hotswap_Hybrid"
+		(property "Footprint" "AlphaCentauri:MX_Choc_Hotswap_Hybrid"
 			(at 297.18 232.41 0)
 			(hide yes)
@@
 			)
 		)
-		(property "Footprint" "JacobGable:MX_Choc_Hotswap_Hybrid_1.5u"
+		(property "Footprint" "AlphaCentauri:MX_Choc_Hotswap_Hybrid_1.5u"
 			(at 240.03 181.61 0)
 			(hide yes)
@@
 			)
 		)
-		(property "Footprint" "JacobGable:MX_Choc_Hotswap_Hybrid"
+		(property "Footprint" "AlphaCentauri:MX_Choc_Hotswap_Hybrid"
 			(at 240.03 207.01 0)
 			(hide yes)
@@
 			)
 		)
-		(property "Footprint" "JacobGable:MX_Choc_Hotswap_Hybrid"
+		(property "Footprint" "AlphaCentauri:MX_Choc_Hotswap_Hybrid"
 			(at 278.13 181.61 0)
 			(hide yes)
@@
 			)
 		)
-		(property "Footprint" "JacobGable:MX_Choc_Hotswap_Hybrid"
+		(property "Footprint" "AlphaCentauri:MX_Choc_Hotswap_Hybrid"
 			(at 278.13 156.21 0)
 			(hide yes)
@@
 			)
 		)
-		(property "Footprint" "JacobGable:MX_Choc_Hotswap_Hybrid"
+		(property "Footprint" "AlphaCentauri:MX_Choc_Hotswap_Hybrid"
 			(at 297.18 156.21 0)
 			(hide yes)
@@
 			)
 		)
-		(property "Footprint" "JacobGable:MX_Choc_Hotswap_Hybrid"
+		(property "Footprint" "AlphaCentauri:MX_Choc_Hotswap_Hybrid"
 			(at 259.08 207.01 0)
 			(hide yes)
@@
 			)
 		)
-		(property "Footprint" "JacobGable:MX_Choc_Hotswap_Hybrid"
+		(property "Footprint" "AlphaCentauri:MX_Choc_Hotswap_Hybrid"
 			(at 335.28 232.41 0)
 			(hide yes)
@@
 			)
 		)
-		(property "Footprint" "JacobGable:MX_Choc_Hotswap_Hybrid"
+		(property "Footprint" "AlphaCentauri:MX_Choc_Hotswap_Hybrid"
 			(at 316.23 232.41 0)
 			(hide yes)
@@
 			)
 		)
-		(property "Footprint" "JacobGable:MX_Choc_Hotswap_Hybrid"
+		(property "Footprint" "AlphaCentauri:MX_Choc_Hotswap_Hybrid"
 			(at 316.23 181.61 0)
 			(hide yes)
@@
 			)
 		)
-		(property "Footprint" "JacobGable:MX_Choc_Hotswap_Hybrid"
+		(property "Footprint" "AlphaCentauri:MX_Choc_Hotswap_Hybrid"
 			(at 316.23 156.21 0)
 			(hide yes)
@@
 			)
 		)
-		(property "Footprint" "JacobGable:MX_Choc_Hotswap_Hybrid"
+		(property "Footprint" "AlphaCentauri:MX_Choc_Hotswap_Hybrid"
 			(at 335.28 207.01 0)
 			(hide yes)
@@
 			)
 		)
-		(property "Footprint" "JacobGable:MX_Choc_Hotswap_Hybrid"
+		(property "Footprint" "AlphaCentauri:MX_Choc_Hotswap_Hybrid"
 			(at 297.18 181.61 0)
 			(hide yes)
@@
 			)
 		)
-		(property "Footprint" "JacobGable:MX_Choc_Hotswap_Hybrid"
+		(property "Footprint" "AlphaCentauri:MX_Choc_Hotswap_Hybrid"
 			(at 278.13 207.01 0)
 			(hide yes)
@@
 			)
 		)
-		(property "Footprint" "JacobGable:MX_Choc_Hotswap_Hybrid"
+		(property "Footprint" "AlphaCentauri:MX_Choc_Hotswap_Hybrid"
 			(at 335.28 181.61 0)
 			(hide yes)
@@
 			)
 		)
-		(property "Footprint" "JacobGable:MX_Choc_Hotswap_Hybrid"
+		(property "Footprint" "AlphaCentauri:MX_Choc_Hotswap_Hybrid"
 			(at 316.23 207.01 0)
 			(hide yes)
@@
 			)
 		)
-		(property "Footprint" "JacobGable:MX_Choc_Hotswap_Hybrid"
+		(property "Footprint" "AlphaCentauri:MX_Choc_Hotswap_Hybrid"
 			(at 259.08 181.61 0)
 			(hide yes)
@@
 			)
 		)
-		(property "Footprint" "JacobGable:MX_Choc_Hotswap_Hybrid"
+		(property "Footprint" "AlphaCentauri:MX_Choc_Hotswap_Hybrid"
 			(at 335.28 156.21 0)
 			(hide yes)
@@
 			)
 		)
-		(property "Footprint" "JacobGable:MX_Choc_Hotswap_Hybrid"
+		(property "Footprint" "AlphaCentauri:MX_Choc_Hotswap_Hybrid"
 			(at 297.18 207.01 0)
 			(hide yes)
