File: pcb/keyboard_r.kicad_sch (KiCad schematic)
At the start: 74 parts, among them J3 USB_C_Receptacle_USB2.0_16P, M5 Motor 1 +, M6 Motor 1 -, M7 Motor 2 +, M8 Motor 2 -, Q2 AO3400A

Commit message: Initial PCB v1.1.0 updates, including 4-layer restructure
Parts:
- added H11: Mounting_Hole, MountingHole:MountingHole_4.3mm_M4, symbol ScottoKeebs:Placeholder_Mounting_Hole
- added S42: SSAG230400, SSAG230400:SSAG230400, symbol SSAG230400:SSAG230400
Connections:
- net 5v R: now also S42.3 (COM); no longer M5.1, M7.1
- new net: M5.1, M7.1, S42.1 (NO_1)
- no-connect marks 5 -> 8
Other:
- moved on the sheet: D54, M5, M6, M7, M8, Q2, R10, R9

Commit message: Include components as a path in the repository
Parts:
- S21, S22, S23, S24, S25, S26, S27, S28, S29, S30, S31, S32, S33, S34, S35, S36, S37, S39, S40: footprint JacobGable:MX_Choc_Hotswap_Hybrid -> AlphaCentauri:MX_Choc_Hotswap_Hybrid
- S38: footprint JacobGable:MX_Choc_Hotswap_Hybrid_1.5u -> AlphaCentauri:MX_Choc_Hotswap_Hybrid_1.5u
Changed lines of the file:
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@@
 			)
 		)
-		(property "Footprint" "JacobGable:MX_Choc_Hotswap_Hybrid"
+		(property "Footprint" "AlphaCentauri:MX_Choc_Hotswap_Hybrid"
 			(at 247.65 231.14 0)
 			(hide yes)
@@
 			)
 		)
-		(property "Footprint" "JacobGable:MX_Choc_Hotswap_Hybrid"
+		(property "Footprint" "AlphaCentauri:MX_Choc_Hotswap_Hybrid"
 			(at 266.7 180.34 0)
 			(hide yes)
@@
 			)
 		)
-		(property "Footprint" "JacobGable:MX_Choc_Hotswap_Hybrid"
+		(property "Footprint" "AlphaCentauri:MX_Choc_Hotswap_Hybrid"
 			(at 304.8 154.94 0)
 			(hide yes)
@@
 			)
 		)
-		(property "Footprint" "JacobGable:MX_Choc_Hotswap_Hybrid"
+		(property "Footprint" "AlphaCentauri:MX_Choc_Hotswap_Hybrid"
 			(at 247.65 154.94 0)
 			(hide yes)
@@
 			)
 		)
-		(property "Footprint" "JacobGable:MX_Choc_Hotswap_Hybrid"
+		(property "Footprint" "AlphaCentauri:MX_Choc_Hotswap_Hybrid"
 			(at 342.9 205.74 0)
 			(hide yes)
@@
 			)
 		)
-		(property "Footprint" "JacobGable:MX_Choc_Hotswap_Hybrid"
+		(property "Footprint" "AlphaCentauri:MX_Choc_Hotswap_Hybrid"
 			(at 285.75 180.34 0)
 			(hide yes)
@@
 			)
 		)
-		(property "Footprint" "JacobGable:MX_Choc_Hotswap_Hybrid"
+		(property "Footprint" "AlphaCentauri:MX_Choc_Hotswap_Hybrid"
 			(at 304.8 180.34 0)
 			(hide yes)
@@
 			)
 		)
-		(property "Footprint" "JacobGable:MX_Choc_Hotswap_Hybrid"
+		(property "Footprint" "AlphaCentauri:MX_Choc_Hotswap_Hybrid"
 			(at 285.75 231.14 0)
 			(hide yes)
@@
 			)
 		)
-		(property "Footprint" "JacobGable:MX_Choc_Hotswap_Hybrid"
+		(property "Footprint" "AlphaCentauri:MX_Choc_Hotswap_Hybrid"
 			(at 266.7 205.74 0)
 			(hide yes)
@@
 			)
 		)
-		(property "Footprint" "JacobGable:MX_Choc_Hotswap_Hybrid"
+		(property "Footprint" "AlphaCentauri:MX_Choc_Hotswap_Hybrid"
 			(at 304.8 205.74 0)
 			(hide yes)
@@
 			)
 		)
-		(property "Footprint" "JacobGable:MX_Choc_Hotswap_Hybrid_1.5u"
+		(property "Footprint" "AlphaCentauri:MX_Choc_Hotswap_Hybrid_1.5u"
 			(at 342.9 180.34 0)
 			(hide yes)
@@
 			)
 		)
-		(property "Footprint" "JacobGable:MX_Choc_Hotswap_Hybrid"
+		(property "Footprint" "AlphaCentauri:MX_Choc_Hotswap_Hybrid"
 			(at 266.7 231.14 0)
 			(hide yes)
@@
 			)
 		)
-		(property "Footprint" "JacobGable:MX_Choc_Hotswap_Hybrid"
+		(property "Footprint" "AlphaCentauri:MX_Choc_Hotswap_Hybrid"
 			(at 323.85 205.74 0)
 			(hide yes)
@@
 			)
 		)
-		(property "Footprint" "JacobGable:MX_Choc_Hotswap_Hybrid"
+		(property "Footprint" "AlphaCentauri:MX_Choc_Hotswap_Hybrid"
 			(at 323.85 180.34 0)
 			(hide yes)
@@
 			)
 		)
-		(property "Footprint" "JacobGable:MX_Choc_Hotswap_Hybrid"
+		(property "Footprint" "AlphaCentauri:MX_Choc_Hotswap_Hybrid"
 			(at 266.7 154.94 0)
 			(hide yes)
@@
 			)
 		)
-		(property "Footprint" "JacobGable:MX_Choc_Hotswap_Hybrid"
+		(property "Footprint" "AlphaCentauri:MX_Choc_Hotswap_Hybrid"
 			(at 285.75 205.74 0)
 			(hide yes)
@@
 			)
 		)
-		(property "Footprint" "JacobGable:MX_Choc_Hotswap_Hybrid"
+		(property "Footprint" "AlphaCentauri:MX_Choc_Hotswap_Hybrid"
 			(at 247.65 180.34 0)
 			(hide yes)
@@
 			)
 		)
-		(property "Footprint" "JacobGable:MX_Choc_Hotswap_Hybrid"
+		(property "Footprint" "AlphaCentauri:MX_Choc_Hotswap_Hybrid"
 			(at 323.85 154.94 0)
 			(hide yes)
@@
 			)
 		)
-		(property "Footprint" "JacobGable:MX_Choc_Hotswap_Hybrid"
+		(property "Footprint" "AlphaCentauri:MX_Choc_Hotswap_Hybrid"
 			(at 285.75 154.94 0)
 			(hide yes)
@@
 			)
 		)
-		(property "Footprint" "JacobGable:MX_Choc_Hotswap_Hybrid"
+		(property "Footprint" "AlphaCentauri:MX_Choc_Hotswap_Hybrid"
 			(at 247.65 205.74 0)
 			(hide yes)
